File: kicad/first-esc/GateDriver.sch (KiCad schematic (older format))
At the start: 30 parts

Commit message: mostly finished schematic, started PCB layout
Parts:
- removed R?: 31k6, symbol Device:R_Small
- removed R?: 0, symbol Device:R_Small
- removed R?: 10k, symbol Device:R_Small
- added R10: 30k, Resistor_SMD:R_0603_1608Metric, symbol Device:R
- added R37: 1k5, Resistor_SMD:R_0603_1608Metric, symbol Device:R
- C1, C12, C14, C16, C17, C2, C3, C4, C5, C6, C7, C8, C9: renamed from C?; footprint (none) -> Capacitor_SMD:C_0603_1608Metric
- C10, C13: renamed from C?; footprint (none) -> Capacitor_SMD:C_1206_3216Metric
- C11, C15: renamed from C?; footprint (none) -> Capacitor_SMD:C_1210_3225Metric
- D1: renamed from D?; value D_Small -> Schottky_100v; footprint (none) -> Diode_SMD:D_SMB
- L1: renamed from L?; footprint (none) -> Inductor_SMD:L_0805_2012Metric
- R11, R4, R5, R6, R7, R8: renamed from R?; footprint (none) -> Resistor_SMD:R_0603_1608Metric
- R9: renamed from R?; value 0 -> 0R; footprint (none) -> Resistor_SMD:R_0603_1608Metric
- U1: renamed from U?; footprint SOP50P810X120-57N -> Package_SO:HTSSOP-56-1EP_6.1x14mm_P0.5mm_EP3.61x6.35mm
Connections:
- net M_OC is gone; now on net +3V3: U1.9 (M_OC)
- net M_PWM is gone; now on net GND: U1.8 (M_PWM)
- net OC_ADJ is gone; now on net DVDD: U1.11 (OC_ADJ)
- net +3V3: now also R10.1, R37.1
- net VSENSE: now also R10.2, R37.2
