File: kicad/first-esc/Power.sch (KiCad schematic (older format))
At the start: 52 parts

Commit message: mostly finished schematic, started PCB layout
Parts:
- C18, C19, C20, C27, C28, C29, C30, C31, C32, C33, C34, C35: renamed from C?; footprint (none) -> Capacitor_SMD:C_0603_1608Metric
- C21, C22, C23, C24, C25, C26: renamed from C?; footprint (none) -> Capacitor_SMD:C_1210_3225Metric
- C36, C37: renamed from C?; footprint (none) -> Capacitor_THT:CP_Radial_D18.0mm_P7.50mm
- Q1, Q2, Q3, Q4, Q5, Q6: renamed from Q?; footprint (none) -> Package_TO_SOT_SMD:TO-252-2
- R12, R13, R14: renamed from R?; footprint (none) -> Resistor_SMD:R_2512_6332Metric; symbol Device:R_Shunt -> Device:R
- R15, R16, R17, R18, R19, R20: renamed from R?; value 4.7R -> 4R7; footprint (none) -> Resistor_SMD:R_0603_1608Metric
- R21, R22, R23: renamed from R?; footprint (none) -> Resistor_SMD:R_0603_1608Metric
- R24, R25, R26, R27, R28, R29, R30, R31: renamed from R?; footprint (none) -> Resistor_SMD:R_0805_2012Metric
- U5, U6, U7: renamed from U?; footprint (none) -> Package_TO_SOT_SMD:SOT-363_SC-70-6
- gave numbers to parts that had none: 3
Connections:
- net PH_A: now also R12.2, U2.3 (-); no longer R12.4
- net PH_B: now also R13.2, U3.3 (-); no longer R13.4
- net PH_C: now also R14.2, U4.3 (-); no longer R14.4
- net SH_A: now also U2.2 (+)
- net SH_B: now also U3.2 (+)
- net SH_C: now also U4.2 (+)
